File: kitt/pcb/mph-pcb/mph-pcb.sch (KiCad schematic (older format))
At the start: 114 parts, among them J1 Screw_Terminal_01x02, J2 Screw_Terminal_01x02, U1 TLC5940NT, U2 TLC5940NT, U3 TLC5940NT, U4 TLC5940NT, U5 TLC5940NT, U6 TLC5940NT, U7 TLC5940NT

Commit message: added msg tx
Parts:
- removed J2: Screw_Terminal_01x02, symbol Connector:Screw_Terminal_01x02
- added J2: Screw_Terminal_01x03, symbol Connector:Screw_Terminal_01x03
Connections:
- net HV_RX: now also J2.2 (Pin_2)
- net HV_TX: now also J2.1 (Pin_1)
- net LV_MSG_TX: now reaches TTGO1.17 (GPIO17)
- net LV_MSG_TX: now also LVL1.8 (LV3)
- net HV_MSG_TX: now reaches LVL1.5 (HV3)
- net HV_MSG_TX: now also J2.3 (Pin_3)
- no-connect marks 32 -> 29
Other:
- moved on the sheet: LVL1

Commit message: add blanking resistors
Parts:
- added R32, R33, R34, R35, R36, R37, R38: 10K, Resistor_THT:R_Axial_DIN0207_L6.3mm_D2.5mm_P10.16mm_Horizontal, symbol Device:R
Connections:
- net +5V: now also R32.1, R33.1, R34.1, R35.1, R36.1, R37.1, R38.1
- net BLANK: now also R32.2, R33.2, R34.2, R35.2, R36.2, R37.2, R38.2
Changed lines of the file:
@@
 	7400 12550 7400 13350
 Wire Wire Line
-	7600 12550 7600 13350
+	7600 12550 7600 12950
 Wire Wire Line
 	7700 12550 7700 13350
@@
 	10000 12550 10000 13350
 Wire Wire Line
-	10200 12550 10200 13350
+	10200 12550 10200 12950
 Wire Wire Line
 	10300 12550 10300 13350
@@
 	12600 12550 12600 13350
 Wire Wire Line
-	12800 12550 12800 13350
+	12800 12550 12800 12950
 Wire Wire Line
 	12900 12550 12900 13350
@@
 	15200 12550 15200 13350
 Wire Wire Line
-	15400 12550 15400 13350
+	15400 12550 15400 12950
 Wire Wire Line
 	15500 12550 15500 13350
@@
 	17800 12550 17800 13350
 Wire Wire Line
-	18000 12550 18000 13350
+	18000 12550 18000 12950
 Wire Wire Line
 	18100 12550 18100 13350
@@
 	20400 12550 20400 13350
 Wire Wire Line
-	20600 12550 20600 13350
+	20600 12550 20600 12950
 Wire Wire Line
 	20700 12550 20700 13350
@@
 	5100 12550 5100 13350
 Wire Wire Line
-	5000 12550 5000 13350
+	5000 12550 5000 12950
 $Comp
 L power:GND #PWR0102
@@
 Wire Wire Line
 	3600 14600 4650 14600
+$Comp
+L Device:R R32
+U 1 1 6113B17E
+P 5350 12950
+F 0 "R32" H 5420 12996 50  0000 L CNN
+F 1 "10K" H 5420 12905 50  0000 L CNN
+F 2 "Resistor_THT:R_Axial_DIN0207_L6.3mm_D2.5mm_P10.16mm_Horizontal" V 5280 12950 50  0001 C CNN
+F 3 "~" H 5350 12950 50  0001 C CNN
+	1    5350 12950
+	0    1    1    0
+$EndComp
+$Comp
+L power:+5V #PWR?
+U 1 1 6116C294
+P 5500 12950
+F 0 "#PWR?" H 5500 12800 50  0001 C CNN
+F 1 "+5V" H 5515 13123 50  0000 C CNN
+F 2 "" H 5500 12950 50  0001 C CNN
+F 3 "" H 5500 12950 50  0001 C CNN
+	1    5500 12950
+	1    0    0    -1
+$EndComp
+Wire Wire Line
+	5200 12950 5000 12950
+Connection ~ 5000 12950
+Wire Wire Line
+	5000 12950 5000 13350
+$Comp
+L Device:R R33
+U 1 1 6119DCC1
+P 7950 12950
+F 0 "R33" H 8020 12996 50  0000 L CNN
+F 1 "10K" H 8020 12905 50  0000 L CNN
+F 2 "Resistor_THT:R_Axial_DIN0207_L6.3mm_D2.5mm_P10.16mm_Horizontal" V 7880 12950 50  0001 C CNN
+F 3 "~" H 7950 12950 50  0001 C CNN
+	1    7950 12950
+	0    1    1    0
+$EndComp
+$Comp
+L power:+5V #PWR?
+U 1 1 6119DCC7
+P 8100 12950
+F 0 "#PWR?" H 8100 12800 50  0001 C CNN
+F 1 "+5V" H 8115 13123 50  0000 C CNN
+F 2 "" H 8100 12950 50  0001 C CNN
+F 3 "" H 8100 12950 50  0001 C CNN
+	1    8100 12950
+	1    0    0    -1
+$EndComp
+Wire Wire Line
+	7800 12950 7600 12950
+Connection ~ 7600 12950
+Wire Wire Line
+	7600 12950 7600 13350
+$Comp
+L Device:R R34
+U 1 1 611FF512
+P 10550 12950
+F 0 "R34" H 10620 12996 50  0000 L CNN
+F 1 "10K" H 10620 12905 50  0000 L CNN
+F 2 "Resistor_THT:R_Axial_DIN0207_L6.3mm_D2.5mm_P10.16mm_Horizontal" V 10480 12950 50  0001 C CNN
+F 3 "~" H 10550 12950 50  0001 C CNN
+	1    10550 12950
+	0    1    1    0
+$EndComp
+$Comp
+L power:+5V #PWR?
+U 1 1 611FF518
+P 10700 12950
+F 0 "#PWR?" H 10700 12800 50  0001 C CNN
+F 1 "+5V" H 10715 13123 50  0000 C CNN
+F 2 "" H 10700 12950 50  0001 C CNN
+F 3 "" H 10700 12950 50  0001 C CNN
+	1    10700 12950
+	1    0    0    -1
+$EndComp
+Wire Wire Line
+	10400 12950 10200 12950
+Connection ~ 10200 12950
+Wire Wire Line
+	10200 12950 10200 13350
+$Comp
+L Device:R R35
+U 1 1 61261A7D
+P 13150 12950
+F 0 "R35" H 13220 12996 50  0000 L CNN
+F 1 "10K" H 13220 12905 50  0000 L CNN
+F 2 "Resistor_THT:R_Axial_DIN0207_L6.3mm_D2.5mm_P10.16mm_Horizontal" V 13080 12950 50  0001 C CNN
+F 3 "~" H 13150 12950 50  0001 C CNN
+	1    13150 12950
+	0    1    1    0
+$EndComp
+$Comp
+L power:+5V #PWR?
+U 1 1 61261A83
+P 13300 12950
+F 0 "#PWR?" H 13300 12800 50  0001 C CNN
+F 1 "+5V" H 13315 13123 50  0000 C CNN
+F 2 "" H 13300 12950 50  0001 C CNN
+F 3 "" H 13300 12950 50  0001 C CNN
+	1    13300 12950
+	1    0    0    -1
+$EndComp
+Wire Wire Line
+	13000 12950 12800 12950
+Connection ~ 12800 12950
+Wire Wire Line
+	12800 12950 12800 13350
+$Comp
+L Device:R R36
+U 1 1 612C4C38
+P 15750 12950
+F 0 "R36" H 15820 12996 50  0000 L CNN
+F 1 "10K" H 15820 12905 50  0000 L CNN
+F 2 "Resistor_THT:R_Axial_DIN0207_L6.3mm_D2.5mm_P10.16mm_Horizontal" V 15680 12950 50  0001 C CNN
+F 3 "~" H 15750 12950 50  0001 C CNN
+	1    15750 12950
+	0    1    1    0
+$EndComp
+$Comp
+L power:+5V #PWR?
+U 1 1 612C4C3E
+P 15900 12950
+F 0 "#PWR?" H 15900 12800 50  0001 C CNN
+F 1 "+5V" H 15915 13123 50  0000 C CNN
+F 2 "" H 15900 12950 50  0001 C CNN
+F 3 "" H 15900 12950 50  0001 C CNN
+	1    15900 12950
+	1    0    0    -1
+$EndComp
+Wire Wire Line
+	15600 12950 15400 12950
+Connection ~ 15400 12950
+Wire Wire Line
+	15400 12950 15400 13350
+$Comp
+L Device:R R37
+U 1 1 61359C5C
+P 18350 12950
+F 0 "R37" H 18420 12996 50  0000 L CNN
+F 1 "10K" H 18420 12905 50  0000 L CNN
+F 2 "Resistor_THT:R_Axial_DIN0207_L6.3mm_D2.5mm_P10.16mm_Horizontal" V 18280 12950 50  0001 C CNN
+F 3 "~" H 18350 12950 50  0001 C CNN
+	1    18350 12950
+	0    1    1    0
+$EndComp
+$Comp
+L power:+5V #PWR?
+U 1 1 61359C62
+P 18500 12950
+F 0 "#PWR?" H 18500 12800 50  0001 C CNN
+F 1 "+5V" H 18515 13123 50  0000 C CNN
+F 2 "" H 18500 12950 50  0001 C CNN
+F 3 "" H 18500 12950 50  0001 C CNN
+	1    18500 12950
+	1    0    0    -1
+$EndComp
+Wire Wire Line
+	18200 12950 18000 12950
+Connection ~ 18000 12950
+Wire Wire Line
+	18000 12950 18000 13350
+$Comp
+L Device:R R38
+U 1 1 613BEB3D
+P 20950 12950
+F 0 "R38" H 21020 12996 50  0000 L CNN
+F 1 "10K" H 21020 12905 50  0000 L CNN
+F 2 "Resistor_THT:R_Axial_DIN0207_L6.3mm_D2.5mm_P10.16mm_Horizontal" V 20880 12950 50  0001 C CNN
+F 3 "~" H 20950 12950 50  0001 C CNN
+	1    20950 12950
+	0    1    1    0
+$EndComp
+$Comp
+L power:+5V #PWR?
+U 1 1 613BEB43
+P 21100 12950
+F 0 "#PWR?" H 21100 12800 50  0001 C CNN
+F 1 "+5V" H 21115 13123 50  0000 C CNN
+F 2 "" H 21100 12950 50  0001 C CNN
+F 3 "" H 21100 12950 50  0001 C CNN
+	1    21100 12950
+	1    0    0    -1
+$EndComp
+Wire Wire Line
+	20800 12950 20600 12950
 Wire Bus Line
 	11650 5050 13500 5050
@@
 Wire Bus Line
 	4400 10250 20700 10250
+Connection ~ 20600 12950
+Wire Wire Line
+	20600 12950 20600 13350
 $EndSCHEMATC

Commit message: copied custom symbols
Parts:
- removed PWR1: OKI-78SR-3.3_1.5-W36H-C, Converter_DCDC:Converter_DCDC_muRata_OKI-78SR_Horizontal, symbol Converter_DCDC:OKI-78SR-3.3_1.5-W36H-C
- added PWR1: OKI-78SR-5_1.5-W36H-C, Converter_DCDC:Converter_DCDC_muRata_OKI-78SR_Horizontal, symbol KITT-Symbols:OKI-78SR-5_1.5-W36H-C
- TTGO1: symbol ttgo_esp32:TTGO_ESP32_TDISPLAY_V1.1 -> KITT-Symbols:TTGO_ESP32_TDISPLAY_V1.1
Connections:
- net +5V: now also PWR1.3 (OUT)
- net GND: now also PWR1.2 (GND)
- net at J1.1 (Pin_1): now also PWR1.1 (IN)
Changed lines of the file:
@@
 $EndComp
 $Comp
-L ttgo_esp32:TTGO_ESP32_TDISPLAY_V1.1 TTGO1
+L KITT-Symbols:TTGO_ESP32_TDISPLAY_V1.1 TTGO1
 U 1 1 610FD390
 P 4850 15350
@@
 HV_RX
 $Comp
-L Converter_DCDC:OKI-78SR-3.3_1.5-W36H-C PWR1
-U 1 1 615C46C8
-P 2800 13250
-F 0 "PWR1" H 2800 13492 50  0000 C CNN
-F 1 "OKI-78SR-3.3_1.5-W36H-C" H 2800 13401 50  0000 C CNN
-F 2 "Converter_DCDC:Converter_DCDC_muRata_OKI-78SR_Horizontal" H 2850 13000 50  0001 L CIN
-F 3 "https://power.murata.com/data/power/oki-78sr.pdf" H 2800 13250 50  0001 C CNN
-	1    2800 13250
-	1    0    0    -1
-$EndComp
-$Comp
 L power:+5V #PWR0150
 U 1 1 61608554
@@
 Wire Wire Line
 	20800 12950 20600 12950
+Connection ~ 20600 12950
+Wire Wire Line
+	20600 12950 20600 13350
 Wire Bus Line
 	11650 5050 13500 5050
@@
 Wire Bus Line
 	4400 10250 20700 10250
-Connection ~ 20600 12950
-Wire Wire Line
-	20600 12950 20600 13350
+$Comp
+L KITT-Symbols:OKI-78SR-5_1.5-W36H-C PWR1
+U 1 1 6117F50F
+P 2800 13250
+F 0 "PWR1" H 2800 13492 50  0000 C CNN
+F 1 "OKI-78SR-5_1.5-W36H-C" H 2800 13401 50  0000 C CNN
+F 2 "Converter_DCDC:Converter_DCDC_muRata_OKI-78SR_Horizontal" H 2850 13000 50  0001 L CIN
+F 3 "https://power.murata.com/data/power/oki-78sr.pdf" H 2800 13250 50  0001 C CNN
+	1    2800 13250
+	1    0    0    -1
+$EndComp
 $EndSCHEMATC

Commit message: fixed typo
Parts:
- renumbered HLT_DISP2 to MASH_DISP2
Changed lines of the file:
@@
 NoConn ~ 4650 14800
 $Comp
-L KITT-Symbols:LDS-A816RI HLT_DISP2
+L KITT-Symbols:LDS-A816RI MASH_DISP2
 U 1 1 6114598A
 P 6250 9000
-F 0 "HLT_DISP2" H 6250 9667 50  0000 C CNN
+F 0 "MASH_DISP2" H 6250 9667 50  0000 C CNN
 F 1 "LDS-A816RI" H 6250 9576 50  0000 C CNN
 F 2 "KITT-Footpads:LDS-A816RI" H 6250 8400 50  0001 C CNN
@@
 Wire Wire Line
 	20600 12950 20600 13350
+$Comp
+L KITT-Symbols:OKI-78SR-5_1.5-W36H-C PWR1
+U 1 1 6117F50F
+P 2800 13250
+F 0 "PWR1" H 2800 13492 50  0000 C CNN
+F 1 "OKI-78SR-5_1.5-W36H-C" H 2800 13401 50  0000 C CNN
+F 2 "Converter_DCDC:Converter_DCDC_muRata_OKI-78SR_Horizontal" H 2850 13000 50  0001 L CIN
+F 3 "https://power.murata.com/data/power/oki-78sr.pdf" H 2800 13250 50  0001 C CNN
+	1    2800 13250
+	1    0    0    -1
+$EndComp
 Wire Bus Line
 	11650 5050 13500 5050
@@
 Wire Bus Line
 	4400 10250 20700 10250
-$Comp
-L KITT-Symbols:OKI-78SR-5_1.5-W36H-C PWR1
-U 1 1 6117F50F
-P 2800 13250
-F 0 "PWR1" H 2800 13492 50  0000 C CNN
-F 1 "OKI-78SR-5_1.5-W36H-C" H 2800 13401 50  0000 C CNN
-F 2 "Converter_DCDC:Converter_DCDC_muRata_OKI-78SR_Horizontal" H 2850 13000 50  0001 L CIN
-F 3 "https://power.murata.com/data/power/oki-78sr.pdf" H 2800 13250 50  0001 C CNN
-	1    2800 13250
-	1    0    0    -1
-$EndComp
 $EndSCHEMATC
