File: kitt/pcb/rpm-pcb/rpm-pcb.sch (KiCad schematic (older format))
At the start: 101 parts, among them J1 Screw_Terminal_01x02, J2 Screw_Terminal_01x03, Q1 NDP6020P, Q2 NDP6020P, Q3 NDP6020P, U1 TLC5940NT, U2 TLC5940NT, U3 TLC5940NT, U4 TLC5940NT, U5 TLC5940NT

Commit message: finished initial wiring
Parts:
- removed HY? (x12): LED, symbol Device:LED
- added LVL2: LVL_5V_3V3, symbol KITT-Symbols:LVL_5V_3V3
- added YD10, YD11, YD12, YD13, YD14, YD15, YD16, YD17, YD18, YD7, YD8, YD9: LED, symbol Device:LED
- gave numbers to parts that had none: 3
- renumbered UG10 to CG10, UG11 to CG11, UG12 to CG12, UG13 to CG13, UG14 to CG14, UG15 to CG15, UG16 to CG16, UG17 to CG17, UG18 to CG18, UG19 to CG19, UG2 to CG2, UG20 to CG20, HT1 to CG21, UG3 to CG3, UG4 to CG4, UG5 to CG5, UG6 to CG6, UG7 to CG7, UG8 to CG8, UG9 to CG9, HT2 to CG_22, HT3 to CG_23, HT4 to CG_24, HT5 to CG_25, HT6 to CG_26, HT7 to CG_27, HT8 to CG_28, HT9 to CG_29, HT10 to CG_30, R32 to R18, R33 to R19, R34 to R20, R35 to R21, R36 to R22, HY1 to YD1, HY2 to YD2, HY3 to YD3
Connections:
- net MASH_DISP3_F is gone; now on net CG_D1: U2.1 (OUT1)
- net SIG_6 is gone; now on net SOUT: U5.17 (SOUT)
- net UG_D1 is gone; now on net KEG_T_L_I: U4.12 (OUT12)
- net UG_YD1 is gone; now on net KEG_T_L_C: U4.6 (OUT6)
- net UG_YD2 is gone; now on net KEG_T_L_D: U4.7 (OUT7)
- net UG_YD3 is gone; now on net KEG_T_L_E: U4.8 (OUT8)
- net UT_YD1 is gone; now on net KEG_T_L_F: U4.9 (OUT9)
- net UT_YD2 is gone; now on net KEG_T_L_G: U4.10 (OUT10)
- net UT_YD3 is gone; now on net KEG_T_L_H: U4.11 (OUT11)
- net +5V: now also LVL2.1 (5V)
- net GND: now also LVL2.11 (GND), LVL2.2 (GND)
- net KEG_1_4_T_ANODE: now also LVL2.5 (HV3)
- net KEG_2_5_T_ANODE: now also LVL2.4 (HV2)
- net at TTGO1.17 (GPIO17): now also LVL2.10 (LV1)
- net at TTGO1.18 (GPIO2): now also LVL2.9 (LV2)
- net at TTGO1.19 (GPIO15): now also LVL2.8 (LV3)
- net at LVL1.12 (3V3), TTGO1.24 (3.3V): now also LVL2.12 (3V3)
- net at KEG_2_T.1 (A), KEG_2_T.11 (F), KEG_2_T.13 (G)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: now also YD10.2 (A), YD11.2 (A), YD12.2 (A), YD7.2 (A), YD8.2 (A), YD9.2 (A)
- net at KEG_3_T.1 (A), KEG_3_T.11 (F), KEG_3_T.13 (G)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: now also YD13.2 (A), YD14.2 (A), YD15.2 (A), YD16.2 (A), YD17.2 (A), YD18.2 (A)
- removed net HLT_YD1: U4.3 (OUT3), YD1.1 (K), YD4.1 (K)
- removed net HLT_YD2: U4.4 (OUT4), YD2.1 (K), YD5.1 (K)
- removed net HLT_YD3: U4.5 (OUT5), YD3.1 (K), YD6.1 (K)
- net HTL_D1: no longer names the net of U3.28 (OUT0)
- net HTL_D1: no longer CG21.1 (K)
- net HTL_D10 renamed CG_D24
- net CG_D24: now also CG_24.1 (K); no longer CG_30.1 (K)
- net HTL_D11 renamed CG_D25
- net CG_D25: now also CG_25.1 (K)
- net HTL_D12 renamed CG_D26
- net CG_D26: now also CG_26.1 (K)
- net HTL_D13 renamed CG_D27
- net CG_D27: now also CG_27.1 (K)
- net HTL_D14 renamed CG_D28
- net CG_D28: now also CG_28.1 (K)
- net HTL_D15 renamed CG_D29
- net CG_D29: now also CG_29.1 (K)
- net HTL_D16 renamed CG_D03
- net HTL_D2 renamed CG_D16
- net CG_D16: now also CG16.1 (K); no longer CG_22.1 (K)
- net HTL_D3 renamed CG_D17
- net CG_D17: now also CG17.1 (K); no longer CG_23.1 (K)
- net HTL_D4 renamed CG_D18
- net CG_D18: now also CG18.1 (K); no longer CG_24.1 (K)
- net HTL_D5 renamed CG_D19
- net CG_D19: now also CG19.1 (K); no longer CG_25.1 (K)
- net HTL_D6 renamed CG_D20
- net CG_D20: now also CG20.1 (K); no longer CG_26.1 (K)
- net HTL_D7 renamed CG_D21
- net CG_D21: now also CG21.1 (K); no longer CG_27.1 (K)
- net HTL_D8 renamed CG_D22
- net CG_D22: now also CG_22.1 (K); no longer CG_28.1 (K)
- net HTL_D9 renamed CG_D23
- net CG_D23: now also CG_23.1 (K); no longer CG_29.1 (K)
- net KEG_1_A renamed KEG_T_L_A
- net KEG_T_L_A: now also U4.4 (OUT4); no longer KEG_4_T.2 (R), KEG_5_T.2 (R), LINE_T.2 (R)
- net KEG_1_B renamed KEG_T_L_B
- net KEG_T_L_B: now also U4.5 (OUT5); no longer KEG_4_T.4 (R), KEG_5_T.4 (R), LINE_T.4 (R)
- net KEG_1_C renamed KEG_T_L_C
- net KEG_T_L_C: no longer KEG_4_T.6 (R), KEG_5_T.6 (R), LINE_T.6 (R)
- net KEG_1_D renamed KEG_T_L_D
- net KEG_T_L_D: no longer KEG_4_T.8 (R), KEG_5_T.8 (R), LINE_T.8 (R)
- net KEG_1_E renamed KEG_T_L_E
- net KEG_T_L_E: no longer KEG_4_T.10 (G), KEG_5_T.10 (G), LINE_T.10 (G)
- net KEG_1_F renamed KEG_T_L_F
- net KEG_T_L_F: no longer KEG_4_T.12 (G), KEG_5_T.12 (G), LINE_T.12 (G)
- net KEG_1_G renamed KEG_T_L_G
- net KEG_T_L_G: no longer KEG_4_T.14 (G), KEG_5_T.14 (G), LINE_T.14 (G)
- net KEG_1_H renamed KEG_T_L_H
- net KEG_T_L_H: no longer KEG_4_T.16 (G), KEG_5_T.16 (G), LINE_T.16 (G)
- net KEG_1_I renamed KEG_T_L_I
- net KEG_T_L_I: no longer KEG_4_T.18 (G), KEG_5_T.18 (G), LINE_T.18 (G)
- net KEG_1_J renamed KEG_T_L_J
- net KEG_T_L_J: now also U4.13 (OUT13); no longer KEG_4_T.20 (G), KEG_5_T.20 (G), LINE_T.20 (G)
- net KEG_1_K renamed KEG_T_L_K
- net KEG_T_L_K: now also U4.14 (OUT14); no longer KEG_4_T.22 (G), KEG_5_T.22 (G), LINE_T.22 (G)
- net KEG_1_L renamed KEG_T_L_L
- net KEG_T_L_L: now also U4.15 (OUT15); no longer KEG_4_T.24 (G), KEG_5_T.24 (G), LINE_T.24 (G)
- net KEG_3_L_T_ANODE renamed KEG_3_L_ANODE
- net KEG_3_L_ANODE: now also LVL2.3 (HV1)
- net MASH_DISP3_A: no longer names the net of U2.28 (OUT0)
- net MASH_DISP3_B renamed CG_D7
- net CG_D7: now also CG7.1 (K)
- net MASH_DISP3_C renamed CG_D5
- net CG_D5: now also CG5.1 (K)
- net MASH_DISP3_D renamed CG_D4
- net CG_D4: now also CG4.1 (K)
- net MASH_DISP3_E renamed CG_D2
- net CG_D2: now also CG2.1 (K)
- net MASH_DISP3_G renamed CG_D6
- net CG_D6: now also CG6.1 (K)
- net MASH_DISP3_RDP renamed CG_D3
- net CG_D3: now also CG3.1 (K)
- net MASH_DISP4_A renamed CG_D8
- net CG_D8: now also CG8.1 (K)
- net MASH_DISP4_B renamed CG_D15
- net CG_D15: now also CG15.1 (K)
- net MASH_DISP4_C renamed CG_D13
- net CG_D13: now also CG13.1 (K)
- net MASH_DISP4_D renamed CG_D12
- net CG_D12: now also CG12.1 (K)
- net MASH_DISP4_E renamed CG_D10
- net CG_D10: now also CG10.1 (K)
- net MASH_DISP4_F renamed CG_D9
- net CG_D9: now also CG9.1 (K)
- net MASH_DISP4_G renamed CG_D14
- net CG_D14: now also CG14.1 (K)
- net MASH_DISP4_RDP renamed CG_D11
- net CG_D11: now also CG11.1 (K)
- net MASH_YD1: no longer names the net of U4.28 (OUT0)
- net MASH_YD2 renamed KEG_T_L_YD1
- net KEG_T_L_YD1: now also YD1.1 (K), YD13.1 (K), YD7.1 (K)
- net MASH_YD3 renamed KEG_T_L_YD2
- net KEG_T_L_YD2: now also YD2.1 (K), YD14.1 (K), YD8.1 (K)
- net UG_D10 renamed KEG_T_R_B
- net KEG_T_R_B: now also KEG_4_T.4 (R), KEG_5_T.4 (R), LINE_T.4 (R); no longer CG10.1 (K)
- net UG_D11 renamed KEG_T_R_C
- net KEG_T_R_C: now also KEG_4_T.6 (R), KEG_5_T.6 (R), LINE_T.6 (R); no longer CG11.1 (K)
- net UG_D12 renamed KEG_T_R_D
- net KEG_T_R_D: now also KEG_4_T.8 (R), KEG_5_T.8 (R), LINE_T.8 (R); no longer CG12.1 (K)
- net UG_D13 renamed KEG_T_R_E
- net KEG_T_R_E: now also KEG_4_T.10 (G), KEG_5_T.10 (G), LINE_T.10 (G); no longer CG13.1 (K)
- net UG_D14 renamed KEG_T_R_F
- net KEG_T_R_F: now also KEG_4_T.12 (G), KEG_5_T.12 (G), LINE_T.12 (G); no longer CG14.1 (K)
- net UG_D15 renamed KEG_T_R_G
- net KEG_T_R_G: now also KEG_4_T.14 (G), KEG_5_T.14 (G), LINE_T.14 (G); no longer CG15.1 (K)
- net UG_D16 renamed KEG_T_R_H
- net KEG_T_R_H: now also KEG_4_T.16 (G), KEG_5_T.16 (G), LINE_T.16 (G); no longer CG16.1 (K)
- net UG_D17 renamed KEG_T_R_I
- net KEG_T_R_I: now also KEG_4_T.18 (G), KEG_5_T.18 (G), LINE_T.18 (G); no longer CG17.1 (K)
- net UG_D18 renamed KEG_T_R_J
- net KEG_T_R_J: now also KEG_4_T.20 (G), KEG_5_T.20 (G), LINE_T.20 (G); no longer CG18.1 (K)
- net UG_D19 renamed KEG_T_R_K
- net KEG_T_R_K: now also KEG_4_T.22 (G), KEG_5_T.22 (G), LINE_T.22 (G); no longer CG19.1 (K)
- removed net UG_D2: CG2.1 (K), U4.13 (OUT13)
- net UG_D20 renamed KEG_T_R_L
- net KEG_T_R_L: now also KEG_4_T.24 (G), KEG_5_T.24 (G), LINE_T.24 (G); no longer CG20.1 (K)
- removed net UG_D3: CG3.1 (K), U4.14 (OUT14)
- removed net UG_D4: CG4.1 (K), U4.15 (OUT15)
- net UG_D5: no longer names the net of U5.28 (OUT0)
- net UG_D5: no longer CG5.1 (K)
- net UG_D6 renamed KEG_T_R_YD1
- net KEG_T_R_YD1: now also YD4.1 (K), YD10.1 (K), YD16.1 (K); no longer CG6.1 (K)
- net UG_D7 renamed KEG_T_R_YD2
- net KEG_T_R_YD2: now also YD5.1 (K), YD11.1 (K), YD17.1 (K); no longer CG7.1 (K)
- net UG_D8 renamed KEG_T_R_YD3
- net KEG_T_R_YD3: no longer CG8.1 (K)
- net UG_D9 renamed KEG_T_R_A
- net KEG_T_R_A: now also KEG_4_T.2 (R), KEG_5_T.2 (R), LINE_T.2 (R); no longer CG9.1 (K)
- new net CG_D30: CG_30.1 (K)
- new net KEG_T_L_YD3: U4.3 (OUT3), YD15.1 (K), YD3.1 (K), YD9.1 (K)
- new net KEG_T_R_YD4: YD12.1 (K), YD18.1 (K), YD6.1 (K)
- no-connect marks 18 -> 21
Other:
- moved on the sheet: J1, J2, LVL1, PWR1, Q1, Q2, Q3

Commit message: fixed for bug checker
Parts:
- renumbered KEG_1_T to KEG_1_T1, KEG_2_T to KEG_2_T1, KEG_3_T to KEG_3_T1, KEG_4_T to KEG_4_T1, KEG_5_T to KEG_5_T1, LINE_T to LINE_T1
Connections:
- net CG_D03 is gone; now on net CG_D30: U3.15 (OUT15)
- net KEG_T_R_YD4 is gone; now on net KEG_T_R_YD3: YD12.1 (K), YD18.1 (K), YD6.1 (K)
Changed lines of the file:
@@
 CG_D29
 Text Label 11050 17700 1    50   ~ 0
-CG_D03
+CG_D30
 Entry Wire Line
 	10800 4550 10900 4450
@@
 Connection ~ 10550 3750
 $Comp
-L KITT-Symbols:STBD01-4R8GA KEG_1_T
+L KITT-Symbols:STBD01-4R8GA KEG_1_T1
 U 1 1 6142D4A0
 P 5350 9250
-F 0 "KEG_1_T" H 6178 9296 50  0000 L CNN
+F 0 "KEG_1_T1" H 6178 9296 50  0000 L CNN
 F 1 "STBD01-4R8GA" H 6178 9205 50  0000 L CNN
 F 2 "" H 4400 9550 50  0001 C CNN
@@
 KEG_T_R_YD2
 Text Label 7850 8250 3    50   ~ 0
-KEG_T_R_YD4
+KEG_T_R_YD3
 Entry Wire Line
 	7400 8850 7500 8750
@@
 	7150 8750 7150 8250
 $Comp
-L KITT-Symbols:STBD01-4R8GA KEG_4_T
+L KITT-Symbols:STBD01-4R8GA KEG_4_T1
 U 1 1 61983C39
 P 8100 9250
-F 0 "KEG_4_T" H 8928 9296 50  0000 L CNN
+F 0 "KEG_4_T1" H 8928 9296 50  0000 L CNN
 F 1 "STBD01-4R8GA" H 8928 9205 50  0000 L CNN
 F 2 "" H 7150 9550 50  0001 C CNN
@@
 	4400 11900 4400 11400
 $Comp
-L KITT-Symbols:STBD01-4R8GA KEG_2_T
+L KITT-Symbols:STBD01-4R8GA KEG_2_T1
 U 1 1 614385DB
 P 5350 12400
-F 0 "KEG_2_T" H 6178 12446 50  0000 L CNN
+F 0 "KEG_2_T1" H 6178 12446 50  0000 L CNN
 F 1 "STBD01-4R8GA" H 6178 12355 50  0000 L CNN
 F 2 "" H 4400 12700 50  0001 C CNN
@@
 KEG_T_R_YD2
 Text Label 7850 11400 3    50   ~ 0
-KEG_T_R_YD4
+KEG_T_R_YD3
 Entry Wire Line
 	7400 12000 7500 11900
@@
 	7150 11900 7150 11400
 $Comp
-L KITT-Symbols:STBD01-4R8GA KEG_5_T
+L KITT-Symbols:STBD01-4R8GA KEG_5_T1
 U 1 1 6143863D
 P 8100 12400
-F 0 "KEG_5_T" H 8928 12446 50  0000 L CNN
+F 0 "KEG_5_T1" H 8928 12446 50  0000 L CNN
 F 1 "STBD01-4R8GA" H 8928 12355 50  0000 L CNN
 F 2 "" H 7150 12700 50  0001 C CNN
@@
 	4400 15150 4400 14650
 $Comp
-L KITT-Symbols:STBD01-4R8GA KEG_3_T
+L KITT-Symbols:STBD01-4R8GA KEG_3_T1
 U 1 1 614E4D99
 P 5350 15650
-F 0 "KEG_3_T" H 6178 15696 50  0000 L CNN
+F 0 "KEG_3_T1" H 6178 15696 50  0000 L CNN
 F 1 "STBD01-4R8GA" H 6178 15605 50  0000 L CNN
 F 2 "" H 4400 15950 50  0001 C CNN
@@
 KEG_T_R_YD2
 Text Label 7850 14650 3    50   ~ 0
-KEG_T_R_YD4
+KEG_T_R_YD3
 Entry Wire Line
 	7400 15250 7500 15150
@@
 	7150 15150 7150 14650
 $Comp
-L KITT-Symbols:STBD01-4R8GA LINE_T
+L KITT-Symbols:STBD01-4R8GA LINE_T1
 U 1 1 614E4DFB
 P 8100 15650
-F 0 "LINE_T" H 8928 15696 50  0000 L CNN
+F 0 "LINE_T1" H 8928 15696 50  0000 L CNN
 F 1 "STBD01-4R8GA" H 8928 15605 50  0000 L CNN
 F 2 "" H 7150 15950 50  0001 C CNN

Commit message: added right bar displays
Parts:
- added C1, C6, C7: 100nF, Capacitor_THT:C_Rect_L7.0mm_W3.5mm_P5.00mm, symbol Device:C
- added C2: 1uF, Capacitor_THT:C_Rect_L7.0mm_W3.5mm_P5.00mm, symbol Device:C
- added J1: Screw_Terminal_01x02, symbol Connector:Screw_Terminal_01x02
- added J2: Screw_Terminal_01x03, symbol Connector:Screw_Terminal_01x03
- added KEG_1_T1, KEG_1_T?, KEG_2_T1, KEG_2_T?, KEG_3_T1, KEG_3_T?, KEG_4_T1, KEG_4_T?, KEG_5_T1, KEG_5_T?, LINE_T1, LINE_T?: STBD01-4R8GA, symbol KITT-Symbols:STBD01-4R8GA
- added LVL1, LVL2: LVL_5V_3V3, symbol KITT-Symbols:LVL_5V_3V3
- added PWR1: OKI-78SR-5_1.5-W36H-C, Converter_DCDC:Converter_DCDC_muRata_OKI-78SR_Horizontal, symbol KITT-Symbols:OKI-78SR-5_1.5-W36H-C
- added Q1, Q2, Q3: NDP6020P, Package_TO_SOT_THT:TO-220-3_Vertical, symbol KITT-Symbols:NDP6020P
- added R23, R26: 2.2K, Resistor_THT:R_Axial_DIN0207_L6.3mm_D2.5mm_P10.16mm_Horizontal, symbol Device:R
- added R24, R26: 10K, Resistor_THT:R_Axial_DIN0207_L6.3mm_D2.5mm_P10.16mm_Horizontal, symbol Device:R
- added TTGO1: TTGO_ESP32_TDISPLAY_V1.1, KITT-Footpads:TTGO_ESP32_TDisplay_v1.1, symbol KITT-Symbols:TTGO_ESP32_TDISPLAY_V1.1
- added U4, U7: TLC5940NT, Package_DIP:DIP-28_W7.62mm, symbol Driver_LED:TLC5940NT
- added YD1, YD10, YD11, YD12, YD13, YD14, YD15, YD16, YD17, YD18, YD2, YD3, YD4, YD5, YD6, YD7, YD8, YD9, YD? (x18): LED, symbol Device:LED
- renumbered C6 to C8, C7 to C9, U4 to U6
Connections:
- net +5V: now also C1.1, C2.1, C6.1, C7.1, LVL1.1 (5V), LVL2.1 (5V), PWR1.3 (OUT), Q1.3 (D), Q2.3 (D), Q3.3 (D), R24.1, R26.1, TTGO1.1 (5V), U4.21 (VCC), U7.21 (VCC)
- net BLANK: now also R24.2, R26.2, TTGO1.3 (GPIO27), U4.23 (BLANK), U7.23 (BLANK)
- net DCPRG: now also TTGO1.10 (GPIO37), TTGO1.9 (GPIO38), U4.19 (DCPRG), U7.19 (DCPRG)
- net GND: now also C1.2, C2.2, C6.2, C7.2, J1.2 (Pin_2), LVL1.11 (GND), LVL1.2 (GND), LVL2.11 (GND), LVL2.2 (GND), PWR1.2 (GND), R23.2, R26.2, TTGO1.13 (GND), TTGO1.14 (GND), TTGO1.2 (GND), TTGO1.22 (GND), TTGO1.23 (GND), U4.22 (GND), U7.22 (GND)
- net GSCLK: now also TTGO1.21 (GPIO12), U4.18 (GSCLK), U7.18 (GSCLK)
- net HV_RX: now also J2.2 (Pin_2), LVL1.4 (HV2)
- net HV_TX: now also J2.1 (Pin_1), LVL1.3 (HV1)
- net KEG_1_4_T_ANODE: now also LVL2.5 (HV3), Q1.1 (G)
- net KEG_2_5_T_ANODE: now also LVL2.4 (HV2), Q2.1 (G)
- net KEG_3_L_ANODE: now also LVL2.3 (HV1), Q3.1 (G)
- net KEG_T_L_A: now also KEG_1_T1.2 (R), KEG_1_T?.2 (R), KEG_2_T1.2 (R), KEG_2_T?.2 (R), KEG_3_T1.2 (R), KEG_3_T?.2 (R), U4.4 (OUT4)
- net KEG_T_L_B: now also KEG_1_T1.4 (R), KEG_1_T?.4 (R), KEG_2_T1.4 (R), KEG_2_T?.4 (R), KEG_3_T1.4 (R), KEG_3_T?.4 (R), U4.5 (OUT5)
- net KEG_T_L_C: now also KEG_1_T1.6 (R), KEG_1_T?.6 (R), KEG_2_T1.6 (R), KEG_2_T?.6 (R), KEG_3_T1.6 (R), KEG_3_T?.6 (R), U4.6 (OUT6)
- net KEG_T_L_D: now also KEG_1_T1.8 (R), KEG_1_T?.8 (R), KEG_2_T1.8 (R), KEG_2_T?.8 (R), KEG_3_T1.8 (R), KEG_3_T?.8 (R), U4.7 (OUT7)
- net KEG_T_L_E: now also KEG_1_T1.10 (G), KEG_1_T?.10 (G), KEG_2_T1.10 (G), KEG_2_T?.10 (G), KEG_3_T1.10 (G), KEG_3_T?.10 (G), U4.8 (OUT8)
- net KEG_T_L_F: now also KEG_1_T1.12 (G), KEG_1_T?.12 (G), KEG_2_T1.12 (G), KEG_2_T?.12 (G), KEG_3_T1.12 (G), KEG_3_T?.12 (G), U4.9 (OUT9)
- net KEG_T_L_G: now also KEG_1_T1.14 (G), KEG_1_T?.14 (G), KEG_2_T1.14 (G), KEG_2_T?.14 (G), KEG_3_T1.14 (G), KEG_3_T?.14 (G), U4.10 (OUT10)
- net KEG_T_L_H: now also KEG_1_T1.16 (G), KEG_1_T?.16 (G), KEG_2_T1.16 (G), KEG_2_T?.16 (G), KEG_3_T1.16 (G), KEG_3_T?.16 (G), U4.11 (OUT11)
- net KEG_T_L_I: now also KEG_1_T1.18 (G), KEG_1_T?.18 (G), KEG_2_T1.18 (G), KEG_2_T?.18 (G), KEG_3_T1.18 (G), KEG_3_T?.18 (G), U4.12 (OUT12)
- net KEG_T_L_J: now also KEG_1_T1.20 (G), KEG_1_T?.20 (G), KEG_2_T1.20 (G), KEG_2_T?.20 (G), KEG_3_T1.20 (G), KEG_3_T?.20 (G), U4.13 (OUT13)
- net KEG_T_L_K: now also KEG_1_T1.22 (G), KEG_1_T?.22 (G), KEG_2_T1.22 (G), KEG_2_T?.22 (G), KEG_3_T1.22 (G), KEG_3_T?.22 (G), U4.14 (OUT14)
- net KEG_T_L_L: now also KEG_1_T1.24 (G), KEG_1_T?.24 (G), KEG_2_T1.24 (G), KEG_2_T?.24 (G), KEG_3_T1.24 (G), KEG_3_T?.24 (G), U4.15 (OUT15)
- net KEG_T_L_YD1: now also U4.1 (OUT1), YD1.1 (K), YD13.1 (K), YD7.1 (K), YD?.1 (K), YD?.1 (K), YD?.1 (K)
- net KEG_T_L_YD2: now also U4.2 (OUT2), YD14.1 (K), YD2.1 (K), YD8.1 (K), YD?.1 (K), YD?.1 (K), YD?.1 (K)
- net KEG_T_L_YD3: now also U4.3 (OUT3), YD15.1 (K), YD3.1 (K), YD9.1 (K), YD?.1 (K), YD?.1 (K), YD?.1 (K)
- net KEG_T_R_A: now also KEG_4_T1.2 (R), KEG_4_T?.2 (R), KEG_5_T1.2 (R), KEG_5_T?.2 (R), LINE_T1.2 (R), LINE_T?.2 (R), U7.4 (OUT4)
- net KEG_T_R_B: now also KEG_4_T1.4 (R), KEG_4_T?.4 (R), KEG_5_T1.4 (R), KEG_5_T?.4 (R), LINE_T1.4 (R), LINE_T?.4 (R), U7.5 (OUT5)
- net KEG_T_R_C: now also KEG_4_T1.6 (R), KEG_4_T?.6 (R), KEG_5_T1.6 (R), KEG_5_T?.6 (R), LINE_T1.6 (R), LINE_T?.6 (R), U7.6 (OUT6)
- net KEG_T_R_D: now also KEG_4_T1.8 (R), KEG_4_T?.8 (R), KEG_5_T1.8 (R), KEG_5_T?.8 (R), LINE_T1.8 (R), LINE_T?.8 (R), U7.7 (OUT7)
- net KEG_T_R_E: now also KEG_4_T1.10 (G), KEG_4_T?.10 (G), KEG_5_T1.10 (G), KEG_5_T?.10 (G), LINE_T1.10 (G), LINE_T?.10 (G), U7.8 (OUT8)
- net KEG_T_R_F: now also KEG_4_T1.12 (G), KEG_4_T?.12 (G), KEG_5_T1.12 (G), KEG_5_T?.12 (G), LINE_T1.12 (G), LINE_T?.12 (G), U7.9 (OUT9)
- net KEG_T_R_G: now also KEG_4_T1.14 (G), KEG_4_T?.14 (G), KEG_5_T1.14 (G), KEG_5_T?.14 (G), LINE_T1.14 (G), LINE_T?.14 (G), U7.10 (OUT10)
- net KEG_T_R_H: now also KEG_4_T1.16 (G), KEG_4_T?.16 (G), KEG_5_T1.16 (G), KEG_5_T?.16 (G), LINE_T1.16 (G), LINE_T?.16 (G), U7.11 (OUT11)
- net KEG_T_R_I: now also KEG_4_T1.18 (G), KEG_4_T?.18 (G), KEG_5_T1.18 (G), KEG_5_T?.18 (G), LINE_T1.18 (G), LINE_T?.18 (G), U7.12 (OUT12)
- net KEG_T_R_J: now also KEG_4_T1.20 (G), KEG_4_T?.20 (G), KEG_5_T1.20 (G), KEG_5_T?.20 (G), LINE_T1.20 (G), LINE_T?.20 (G), U7.13 (OUT13)
- net KEG_T_R_K: now also KEG_4_T1.22 (G), KEG_4_T?.22 (G), KEG_5_T1.22 (G), KEG_5_T?.22 (G), LINE_T1.22 (G), LINE_T?.22 (G), U7.14 (OUT14)
- net KEG_T_R_L: now also KEG_4_T1.24 (G), KEG_4_T?.24 (G), KEG_5_T1.24 (G), KEG_5_T?.24 (G), LINE_T1.24 (G), LINE_T?.24 (G), U7.15 (OUT15)
- net KEG_T_R_YD1: now also U7.1 (OUT1), YD10.1 (K), YD16.1 (K), YD4.1 (K), YD?.1 (K), YD?.1 (K), YD?.1 (K)
- net KEG_T_R_YD2: now also U7.2 (OUT2), YD11.1 (K), YD17.1 (K), YD5.1 (K), YD?.1 (K), YD?.1 (K), YD?.1 (K)
- net KEG_T_R_YD3: now also U7.3 (OUT3), YD12.1 (K), YD18.1 (K), YD6.1 (K), YD?.1 (K), YD?.1 (K), YD?.1 (K)
- net LV_RX: now also LVL1.9 (LV2), TTGO1.16 (GPIO22)
- net LV_TX: now also LVL1.10 (LV1), TTGO1.15 (GPIO21)
- net SCLK: now also TTGO1.5 (GPIO25), U4.25 (SCLK), U7.25 (SCLK)
- net SIG_1: now also TTGO1.6 (GPIO33)
- net SIG_4: now also U4.26 (SIN)
- net SIG_5: now also U4.17 (SOUT), U7.26 (SIN)
- net SOUT: now also TTGO1.20 (GPIO13), U7.17 (SOUT)
- net VPRG: now also TTGO1.7 (GPIO32), U4.27 (VPRG), U7.27 (VPRG)
- net XLAT: now also TTGO1.4 (GPIO26), U4.24 (XLAT), U7.24 (XLAT)
- net at LVL2.12 (3V3), TTGO1.24 (3.3V): now also LVL1.12 (3V3); no longer LVL1.12 (3V3)
- net at U6.20 (IREF): now also R23.1; no longer R4.1
- net at KEG_1_T1.1 (A), KEG_1_T1.11 (F), KEG_1_T1.13 (G)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: now also KEG_1_T?.1 (A), KEG_1_T?.11 (F), KEG_1_T?.13 (G), KEG_1_T?.15 (H), KEG_1_T?.17 (I), KEG_1_T?.19 (J), KEG_1_T?.21 (K), KEG_1_T?.23 (L), KEG_1_T?.3 (B), KEG_1_T?.5 (C), KEG_1_T?.7 (D), KEG_1_T?.9 (E), KEG_4_T?.1 (A), KEG_4_T?.11 (F), KEG_4_T?.13 (G), KEG_4_T?.15 (H), KEG_4_T?.17 (I), KEG_4_T?.19 (J), KEG_4_T?.21 (K), KEG_4_T?.23 (L), KEG_4_T?.3 (B), KEG_4_T?.5 (C), KEG_4_T?.7 (D), KEG_4_T?.9 (E), Q1.2 (S), YD5.2 (A), YD?.2 (A), YD?.2 (A), YD?.2 (A), YD?.2 (A), YD?.2 (A), YD?.2 (A); no longer Q1.2 (S), YD5.2 (A)
- net at KEG_2_T1.1 (A), KEG_2_T1.11 (F), KEG_2_T1.13 (G)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: now also YD10.2 (A), YD11.2 (A), YD12.2 (A); no longer YD10.2 (A), YD11.2 (A), YD12.2 (A)
- net at KEG_3_T1.1 (A), KEG_3_T1.11 (F), KEG_3_T1.13 (G)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: now also KEG_3_T?.1 (A), KEG_3_T?.11 (F), KEG_3_T?.13 (G), KEG_3_T?.15 (H), KEG_3_T?.17 (I), KEG_3_T?.19 (J), KEG_3_T?.21 (K), KEG_3_T?.23 (L), KEG_3_T?.3 (B), KEG_3_T?.5 (C), KEG_3_T?.7 (D), KEG_3_T?.9 (E), LINE_T?.1 (A), LINE_T?.11 (F), LINE_T?.13 (G), LINE_T?.15 (H), LINE_T?.17 (I), LINE_T?.19 (J), LINE_T?.21 (K), LINE_T?.23 (L), LINE_T?.3 (B), LINE_T?.5 (C), LINE_T?.7 (D), LINE_T?.9 (E), Q3.2 (S), YD13.2 (A), YD16.2 (A), YD?.2 (A), YD?.2 (A), YD?.2 (A), YD?.2 (A), YD?.2 (A), YD?.2 (A); no longer Q3.2 (S), YD13.2 (A), YD16.2 (A)
- new net: R4.1, U4.20 (IREF)
- new net: LVL2.10 (LV1), TTGO1.17 (GPIO17)
- new net: LVL2.9 (LV2), TTGO1.18 (GPIO2)
- new net: LVL2.8 (LV3), TTGO1.19 (GPIO15)
- new net: LVL1.12 (3V3), LVL2.12 (3V3), TTGO1.24 (3.3V)
- new net: J1.1 (Pin_1), PWR1.1 (IN)
- new net: R26.1, U7.20 (IREF)
- new net: KEG_1_T1.1 (A), KEG_1_T1.11 (F), KEG_1_T1.13 (G), KEG_1_T1.15 (H), KEG_1_T1.17 (I), KEG_1_T1.19 (J), KEG_1_T1.21 (K), KEG_1_T1.23 (L), KEG_1_T1.3 (B), KEG_1_T1.5 (C), KEG_1_T1.7 (D), KEG_1_T1.9 (E), KEG_4_T1.1 (A), KEG_4_T1.11 (F), KEG_4_T1.13 (G), KEG_4_T1.15 (H), KEG_4_T1.17 (I), KEG_4_T1.19 (J), KEG_4_T1.21 (K), KEG_4_T1.23 (L), KEG_4_T1.3 (B), KEG_4_T1.5 (C), KEG_4_T1.7 (D), KEG_4_T1.9 (E), Q1.2 (S), YD1.2 (A), YD2.2 (A), YD3.2 (A), YD4.2 (A), YD5.2 (A), YD6.2 (A)
- new net: KEG_2_T1.1 (A), KEG_2_T1.11 (F), KEG_2_T1.13 (G), KEG_2_T1.15 (H), KEG_2_T1.17 (I), KEG_2_T1.19 (J), KEG_2_T1.21 (K), KEG_2_T1.23 (L), KEG_2_T1.3 (B), KEG_2_T1.5 (C), KEG_2_T1.7 (D), KEG_2_T1.9 (E), KEG_2_T?.1 (A), KEG_2_T?.11 (F), KEG_2_T?.13 (G), KEG_2_T?.15 (H), KEG_2_T?.17 (I), KEG_2_T?.19 (J), KEG_2_T?.21 (K), KEG_2_T?.23 (L), KEG_2_T?.3 (B), KEG_2_T?.5 (C), KEG_2_T?.7 (D), KEG_2_T?.9 (E), KEG_5_T1.1 (A), KEG_5_T1.11 (F), KEG_5_T1.13 (G), KEG_5_T1.15 (H), KEG_5_T1.17 (I), KEG_5_T1.19 (J), KEG_5_T1.21 (K), KEG_5_T1.23 (L), KEG_5_T1.3 (B), KEG_5_T1.5 (C), KEG_5_T1.7 (D), KEG_5_T1.9 (E), KEG_5_T?.1 (A), KEG_5_T?.11 (F), KEG_5_T?.13 (G), KEG_5_T?.15 (H), KEG_5_T?.17 (I), KEG_5_T?.19 (J), KEG_5_T?.21 (K), KEG_5_T?.23 (L), KEG_5_T?.3 (B), KEG_5_T?.5 (C), KEG_5_T?.7 (D), KEG_5_T?.9 (E), Q2.2 (S), YD10.2 (A), YD11.2 (A), YD12.2 (A), YD7.2 (A), YD8.2 (A), YD9.2 (A), YD?.2 (A), YD?.2 (A), YD?.2 (A), YD?.2 (A), YD?.2 (A), YD?.2 (A)
- new net: KEG_3_T1.1 (A), KEG_3_T1.11 (F), KEG_3_T1.13 (G), KEG_3_T1.15 (H), KEG_3_T1.17 (I), KEG_3_T1.19 (J), KEG_3_T1.21 (K), KEG_3_T1.23 (L), KEG_3_T1.3 (B), KEG_3_T1.5 (C), KEG_3_T1.7 (D), KEG_3_T1.9 (E), LINE_T1.1 (A), LINE_T1.11 (F), LINE_T1.13 (G), LINE_T1.15 (H), LINE_T1.17 (I), LINE_T1.19 (J), LINE_T1.21 (K), LINE_T1.23 (L), LINE_T1.3 (B), LINE_T1.5 (C), LINE_T1.7 (D), LINE_T1.9 (E), Q3.2 (S), YD13.2 (A), YD14.2 (A), YD15.2 (A), YD16.2 (A), YD17.2 (A), YD18.2 (A)
- no-connect marks 21 -> 35
Other:
- moved on the sheet: C1, C2, C3, C8, C9, CG1, CG10, CG11, CG12, CG13, CG14, CG15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

Commit message: finished wiring and bug check
Parts:
- removed J1: Screw_Terminal_01x02, symbol Connector:Screw_Terminal_01x02
- removed J2: Screw_Terminal_01x03, symbol Connector:Screw_Terminal_01x03
- removed LVL1: LVL_5V_3V3, symbol KITT-Symbols:LVL_5V_3V3
- removed PWR1: OKI-78SR-5_1.5-W36H-C, Converter_DCDC:Converter_DCDC_muRata_OKI-78SR_Horizontal, symbol KITT-Symbols:OKI-78SR-5_1.5-W36H-C
- removed YD10, YD11, YD12, YD16, YD17, YD18, YD4, YD5, YD6, YD? (x9): LED, symbol Device:LED
- added C10, C11: 100nF, Capacitor_THT:C_Rect_L7.0mm_W3.5mm_P5.00mm, symbol Device:C
- added R27, R29: 2.2K, Resistor_THT:R_Axial_DIN0207_L6.3mm_D2.5mm_P10.16mm_Horizontal, symbol Device:R
- added R28, R30: 10K, Resistor_THT:R_Axial_DIN0207_L6.3mm_D2.5mm_P10.16mm_Horizontal, symbol Device:R
- added U8, U9: TLC5940NT, Package_DIP:DIP-28_W7.62mm, symbol Driver_LED:TLC5940NT
- gave numbers to parts that had none: 15
- renumbered C1 to C12, C2 to C13, KEG_1_T1 to LAGER_1_T_L1, KEG_4_T1 to LAGER_1_T_R1, KEG_2_T1 to LAGER_2_T_L1, KEG_5_T1 to LAGER_2_T_R1, KEG_3_T1 to LAGER_3_T_L1, LINE_T1 to LAGER_3_T_R1, LVL2 to LVL3, Q1 to Q4, Q2 to Q5, Q3 to Q6, R26 to R25, TTGO1 to TTGO2, YD1 to YD19, YD2 to YD20, YD3 to YD21, YD7 to YD25, YD8 to YD26, YD9 to YD27, YD13 to YD31, YD14 to YD32, YD15 to YD33
Connections:
- net +5V: now also C10.1, C11.1, R28.1, R30.1, U8.21 (VCC), U9.21 (VCC)
- net BLANK: no longer R24.2, R26.2, TTGO2.3 (GPIO27), U6.23 (BLANK), U7.23 (BLANK)
- net DCPRG: no longer TTGO2.10 (GPIO37), TTGO2.9 (GPIO38), U6.19 (DCPRG), U7.19 (DCPRG)
- net GND: now also C10.2, C11.2, R27.2, R29.2, U8.22 (GND), U9.22 (GND)
- net GSCLK: no longer TTGO2.21 (GPIO12), U6.18 (GSCLK), U7.18 (GSCLK)
- net KEG_T_L_A: no longer KEG_1_CAP_L1.2 (R), KEG_CAP_2_L1.2 (R), KEG_CAP_3_L1.2 (R), LAGER_1_T_L1.2 (R), LAGER_2_T_L1.2 (R), LAGER_3_T_L1.2 (R), U6.4 (OUT4)
- net KEG_T_L_B: no longer KEG_1_CAP_L1.4 (R), KEG_CAP_2_L1.4 (R), KEG_CAP_3_L1.4 (R), LAGER_1_T_L1.4 (R), LAGER_2_T_L1.4 (R), LAGER_3_T_L1.4 (R), U6.5 (OUT5)
- net KEG_T_L_C: no longer KEG_1_CAP_L1.6 (R), KEG_CAP_2_L1.6 (R), KEG_CAP_3_L1.6 (R), LAGER_1_T_L1.6 (R), LAGER_2_T_L1.6 (R), LAGER_3_T_L1.6 (R), U6.6 (OUT6)
- net KEG_T_L_D: no longer KEG_1_CAP_L1.8 (R), KEG_CAP_2_L1.8 (R), KEG_CAP_3_L1.8 (R), LAGER_1_T_L1.8 (R), LAGER_2_T_L1.8 (R), LAGER_3_T_L1.8 (R), U6.7 (OUT7)
- net KEG_T_L_E: no longer KEG_1_CAP_L1.10 (G), KEG_CAP_2_L1.10 (G), KEG_CAP_3_L1.10 (G), LAGER_1_T_L1.10 (G), LAGER_2_T_L1.10 (G), LAGER_3_T_L1.10 (G), U6.8 (OUT8)
- net KEG_T_L_F: no longer KEG_1_CAP_L1.12 (G), KEG_CAP_2_L1.12 (G), KEG_CAP_3_L1.12 (G), LAGER_1_T_L1.12 (G), LAGER_2_T_L1.12 (G), LAGER_3_T_L1.12 (G), U6.9 (OUT9)
- net KEG_T_L_G: no longer KEG_1_CAP_L1.14 (G), KEG_CAP_2_L1.14 (G), KEG_CAP_3_L1.14 (G), LAGER_1_T_L1.14 (G), LAGER_2_T_L1.14 (G), LAGER_3_T_L1.14 (G), U6.10 (OUT10)
- net KEG_T_L_H: no longer KEG_1_CAP_L1.16 (G), KEG_CAP_2_L1.16 (G), KEG_CAP_3_L1.16 (G), LAGER_1_T_L1.16 (G), LAGER_2_T_L1.16 (G), LAGER_3_T_L1.16 (G), U6.11 (OUT11)
- net KEG_T_L_I: no longer KEG_1_CAP_L1.18 (G), KEG_CAP_2_L1.18 (G), KEG_CAP_3_L1.18 (G), LAGER_1_T_L1.18 (G), LAGER_2_T_L1.18 (G), LAGER_3_T_L1.18 (G), U6.12 (OUT12)
- net KEG_T_L_J: no longer KEG_1_CAP_L1.20 (G), KEG_CAP_2_L1.20 (G), KEG_CAP_3_L1.20 (G), LAGER_1_T_L1.20 (G), LAGER_2_T_L1.20 (G), LAGER_3_T_L1.20 (G), U6.13 (OUT13)
- net KEG_T_L_K: no longer KEG_1_CAP_L1.22 (G), KEG_CAP_2_L1.22 (G), KEG_CAP_3_L1.22 (G), LAGER_1_T_L1.22 (G), LAGER_2_T_L1.22 (G), LAGER_3_T_L1.22 (G), U6.14 (OUT14)
- net KEG_T_L_L: no longer KEG_1_CAP_L1.24 (G), KEG_CAP_2_L1.24 (G), KEG_CAP_3_L1.24 (G), LAGER_1_T_L1.24 (G), LAGER_2_T_L1.24 (G), LAGER_3_T_L1.24 (G), U6.15 (OUT15)
- net KEG_T_L_YD1: no longer U6.1 (OUT1), YD19.1 (K), YD25.1 (K), YD31.1 (K), YD37.1 (K), YD43.1 (K), YD49.1 (K)
- net KEG_T_L_YD2: no longer U6.2 (OUT2), YD26.1 (K), YD32.1 (K), YD38.1 (K), YD44.1 (K), YD50.1 (K)
- net KEG_T_L_YD3: no longer U6.3 (OUT3), YD27.1 (K), YD33.1 (K), YD39.1 (K), YD45.1 (K), YD51.1 (K)
- net KEG_T_R_A: no longer KEG_1_CAP_R1.2 (R), KEG_CAP_2_R1.2 (R), KEG_CAP_3_R1.2 (R), LAGER_1_T_R1.2 (R), LAGER_2_T_R1.2 (R), LAGER_3_T_R1.2 (R), U7.4 (OUT4)
- net KEG_T_R_B: no longer KEG_1_CAP_R1.4 (R), KEG_CAP_2_R1.4 (R), KEG_CAP_3_R1.4 (R), LAGER_1_T_R1.4 (R), LAGER_2_T_R1.4 (R), LAGER_3_T_R1.4 (R), U7.5 (OUT5)
- net KEG_T_R_C: no longer KEG_1_CAP_R1.6 (R), KEG_CAP_2_R1.6 (R), KEG_CAP_3_R1.6 (R), LAGER_1_T_R1.6 (R), LAGER_2_T_R1.6 (R), LAGER_3_T_R1.6 (R), U7.6 (OUT6)
- net KEG_T_R_D: no longer KEG_1_CAP_R1.8 (R), KEG_CAP_2_R1.8 (R), KEG_CAP_3_R1.8 (R), LAGER_1_T_R1.8 (R), LAGER_2_T_R1.8 (R), LAGER_3_T_R1.8 (R), U7.7 (OUT7)
- net KEG_T_R_E: no longer KEG_1_CAP_R1.10 (G), KEG_CAP_2_R1.10 (G), KEG_CAP_3_R1.10 (G), LAGER_1_T_R1.10 (G), LAGER_2_T_R1.10 (G), LAGER_3_T_R1.10 (G), U7.8 (OUT8)
- net KEG_T_R_F: no longer KEG_1_CAP_R1.12 (G), KEG_CAP_2_R1.12 (G), KEG_CAP_3_R1.12 (G), LAGER_1_T_R1.12 (G), LAGER_2_T_R1.12 (G), LAGER_3_T_R1.12 (G)
- net KEG_T_R_G: no longer KEG_1_CAP_R1.14 (G), KEG_CAP_2_R1.14 (G), KEG_CAP_3_R1.14 (G), LAGER_1_T_R1.14 (G), LAGER_2_T_R1.14 (G), LAGER_3_T_R1.14 (G)
- net KEG_T_R_H: no longer KEG_1_CAP_R1.16 (G), KEG_CAP_2_R1.16 (G), KEG_CAP_3_R1.16 (G), LAGER_1_T_R1.16 (G), LAGER_2_T_R1.16 (G), LAGER_3_T_R1.16 (G)
- net KEG_T_R_I: no longer KEG_1_CAP_R1.18 (G), KEG_CAP_2_R1.18 (G), KEG_CAP_3_R1.18 (G), LAGER_1_T_R1.18 (G), LAGER_2_T_R1.18 (G), LAGER_3_T_R1.18 (G)
- net KEG_T_R_J: no longer KEG_1_CAP_R1.20 (G), KEG_CAP_2_R1.20 (G), KEG_CAP_3_R1.20 (G), LAGER_1_T_R1.20 (G), LAGER_2_T_R1.20 (G), LAGER_3_T_R1.20 (G)
- net KEG_T_R_K: no longer KEG_1_CAP_R1.22 (G), KEG_CAP_2_R1.22 (G), KEG_CAP_3_R1.22 (G), LAGER_1_T_R1.22 (G), LAGER_2_T_R1.22 (G), LAGER_3_T_R1.22 (G)
- net KEG_T_R_L: no longer KEG_1_CAP_R1.24 (G), KEG_CAP_2_R1.24 (G), KEG_CAP_3_R1.24 (G), LAGER_1_T_R1.24 (G), LAGER_2_T_R1.24 (G), LAGER_3_T_R1.24 (G)
- net KEG_T_R_YD1: no longer U7.1 (OUT1)
- net KEG_T_R_YD2: no longer U7.2 (OUT2)
- net KEG_T_R_YD3: no longer U7.3 (OUT3)
- net LV_RX: no longer TTGO2.16 (GPIO22)
- net LV_TX: no longer TTGO2.15 (GPIO21)
- net SCLK: no longer TTGO2.5 (GPIO25), U6.25 (SCLK), U7.25 (SCLK)
- net SIG_1: no longer TTGO2.6 (GPIO33)
- net SIG_4: no longer U6.26 (SIN)
- net SIG_5: no longer U6.17 (SOUT), U7.26 (SIN)
- net SOUT: no longer TTGO2.20 (GPIO13), U7.17 (SOUT)
- net VPRG: no longer TTGO2.7 (GPIO32), U6.27 (VPRG), U7.27 (VPRG)
- net XLAT: no longer TTGO2.4 (GPIO26), U6.24 (XLAT), U7.24 (XLAT)
- net KEG_1_4_T_ANODE: no longer names the net of LVL3.5 (HV3), Q4.1 (G)
- net KEG_1_4_T_ANODE: no longer LVL2.5 (HV3), Q1.1 (G)
- net KEG_2_5_T_ANODE: no longer names the net of LVL2.4 (HV2), Q2.1 (G)
- net KEG_2_5_T_ANODE: no longer LVL3.4 (HV2), Q5.1 (G)
- net KEG_3_L_ANODE: no longer names the net of LVL2.3 (HV1), Q3.1 (G)
- net KEG_3_L_ANODE: no longer LVL3.3 (HV1), Q6.1 (G)
- new net: LVL2.5 (HV3), Q1.1 (G)
- new net: LVL3.4 (HV2), Q5.1 (G)
- new net: LVL3.3 (HV1), Q6.1 (G)
- new net: R27.1, U8.20 (IREF)
- new net: R29.1, U9.20 (IREF)
- new net BLANK_2: R24.2, R26.2, R28.2, R30.2, TTGO2.3 (GPIO27), U6.23 (BLANK), U7.23 (BLANK), U8.23 (BLANK), U9.23 (BLANK)
- new net DCPRG_2: TTGO2.10 (GPIO37), TTGO2.9 (GPIO38), U6.19 (DCPRG), U7.19 (DCPRG), U8.19 (DCPRG), U9.19 (DCPRG)
- new net GSCLK_2: TTGO2.21 (GPIO12), U6.18 (GSCLK), U7.18 (GSCLK), U8.18 (GSCLK), U9.18 (GSCLK)
- new net KEG_CAP_L_A: KEG_1_CAP_L1.2 (R), KEG_CAP_2_L1.2 (R), KEG_CAP_3_L1.2 (R), U8.4 (OUT4)
- new net KEG_CAP_L_B: KEG_1_CAP_L1.4 (R), KEG_CAP_2_L1.4 (R), KEG_CAP_3_L1.4 (R), U8.5 (OUT5)
- new net KEG_CAP_L_C: KEG_1_CAP_L1.6 (R), KEG_CAP_2_L1.6 (R), KEG_CAP_3_L1.6 (R), U8.6 (OUT6)
- new net KEG_CAP_L_D: KEG_1_CAP_L1.8 (R), KEG_CAP_2_L1.8 (R), KEG_CAP_3_L1.8 (R), U8.7 (OUT7)
- new net KEG_CAP_L_E: KEG_1_CAP_L1.10 (G), KEG_CAP_2_L1.10 (G), KEG_CAP_3_L1.10 (G), U8.8 (OUT8)
- new net KEG_CAP_L_F: KEG_1_CAP_L1.12 (G), KEG_CAP_2_L1.12 (G), KEG_CAP_3_L1.12 (G), U8.9 (OUT9)
- new net KEG_CAP_L_G: KEG_1_CAP_L1.14 (G), KEG_CAP_2_L1.14 (G), KEG_CAP_3_L1.14 (G), U8.10 (OUT10)
- new net KEG_CAP_L_H: KEG_1_CAP_L1.16 (G), KEG_CAP_2_L1.16 (G), KEG_CAP_3_L1.16 (G), U8.11 (OUT11)
- new net KEG_CAP_L_I: KEG_1_CAP_L1.18 (G), KEG_CAP_2_L1.18 (G), KEG_CAP_3_L1.18 (G), U8.12 (OUT12)
- new net KEG_CAP_L_J: KEG_1_CAP_L1.20 (G), KEG_CAP_2_L1.20 (G), KEG_CAP_3_L1.20 (G), U8.13 (OUT13)
- new net KEG_CAP_L_K: KEG_1_CAP_L1.22 (G), KEG_CAP_2_L1.22 (G), KEG_CAP_3_L1.22 (G), U8.14 (OUT14)
- new net KEG_CAP_L_L: KEG_1_CAP_L1.24 (G), KEG_CAP_2_L1.24 (G), KEG_CAP_3_L1.24 (G), U8.15 (OUT15)
- new net KEG_CAP_L_YD1: U8.1 (OUT1), YD37.1 (K), YD43.1 (K), YD49.1 (K)
- new net KEG_CAP_L_YD2: U8.2 (OUT2), YD38.1 (K), YD44.1 (K), YD50.1 (K)
- new net KEG_CAP_L_YD3: U8.3 (OUT3), YD39.1 (K), YD45.1 (K), YD51.1 (K)
- new net KEG_CAP_R_A: KEG_1_CAP_R1.2 (R), KEG_CAP_2_R1.2 (R), KEG_CAP_3_R1.2 (R), U9.4 (OUT4)
- new net KEG_CAP_R_B: KEG_1_CAP_R1.4 (R), KEG_CAP_2_R1.4 (R), KEG_CAP_3_R1.4 (R), U9.5 (OUT5)
- new net KEG_CAP_R_C: KEG_1_CAP_R1.6 (R), KEG_CAP_2_R1.6 (R), KEG_CAP_3_R1.6 (R), U9.6 (OUT6)
- new net KEG_CAP_R_D: KEG_1_CAP_R1.8 (R), KEG_CAP_2_R1.8 (R), KEG_CAP_3_R1.8 (R), U9.7 (OUT7)
- new net KEG_CAP_R_E: KEG_1_CAP_R1.10 (G), KEG_CAP_2_R1.10 (G), KEG_CAP_3_R1.10 (G), U9.8 (OUT8)
- new net KEG_CAP_R_F: KEG_1_CAP_R1.12 (G), KEG_CAP_2_R1.12 (G), KEG_CAP_3_R1.12 (G), U9.9 (OUT9)
- new net KEG_CAP_R_G: KEG_1_CAP_R1.14 (G), KEG_CAP_2_R1.14 (G), KEG_CAP_3_R1.14 (G), U9.10 (OUT10)
- new net KEG_CAP_R_H: KEG_1_CAP_R1.16 (G), KEG_CAP_2_R1.16 (G), KEG_CAP_3_R1.16 (G), U9.11 (OUT11)
- new net KEG_CAP_R_I: KEG_1_CAP_R1.18 (G), KEG_CAP_2_R1.18 (G), KEG_CAP_3_R1.18 (G), U9.12 (OUT12)
- new net KEG_CAP_R_J: KEG_1_CAP_R1.20 (G), KEG_CAP_2_R1.20 (G), KEG_CAP_3_R1.20 (G), U9.13 (OUT13)
- new net KEG_CAP_R_K: KEG_1_CAP_R1.22 (G), KEG_CAP_2_R1.22 (G), KEG_CAP_3_R1.22 (G), U9.14 (OUT14)
- new net KEG_CAP_R_L: KEG_1_CAP_R1.24 (G), KEG_CAP_2_R1.24 (G), KEG_CAP_3_R1.24 (G), U9.15 (OUT15)
- new net LAGER_L_A: LAGER_1_T_L1.2 (R), LAGER_2_T_L1.2 (R), LAGER_3_T_L1.2 (R), U6.4 (OUT4)
- new net LAGER_L_B: LAGER_1_T_L1.4 (R), LAGER_2_T_L1.4 (R), LAGER_3_T_L1.4 (R), U6.5 (OUT5)
- new net LAGER_L_C: LAGER_1_T_L1.6 (R), LAGER_2_T_L1.6 (R), LAGER_3_T_L1.6 (R), U6.6 (OUT6)
- new net LAGER_L_D: LAGER_1_T_L1.8 (R), LAGER_2_T_L1.8 (R), LAGER_3_T_L1.8 (R), U6.7 (OUT7)
- new net LAGER_L_E: LAGER_1_T_L1.10 (G), LAGER_2_T_L1.10 (G), LAGER_3_T_L1.10 (G), U6.8 (OUT8)
- new net LAGER_L_F: LAGER_1_T_L1.12 (G), LAGER_2_T_L1.12 (G), LAGER_3_T_L1.12 (G), U6.9 (OUT9)
- new net LAGER_L_G: LAGER_1_T_L1.14 (G), LAGER_2_T_L1.14 (G), LAGER_3_T_L1.14 (G), U6.10 (OUT10)
- new net LAGER_L_H: LAGER_1_T_L1.16 (G), LAGER_2_T_L1.16 (G), LAGER_3_T_L1.16 (G), U6.11 (OUT11)
- new net LAGER_L_I: LAGER_1_T_L1.18 (G), LAGER_2_T_L1.18 (G), LAGER_3_T_L1.18 (G), U6.12 (OUT12)
- new net LAGER_L_J: LAGER_1_T_L1.20 (G), LAGER_2_T_L1.20 (G), LAGER_3_T_L1.20 (G), U6.13 (OUT13)
- new net LAGER_L_K: LAGER_1_T_L1.22 (G), LAGER_2_T_L1.22 (G), LAGER_3_T_L1.22 (G), U6.14 (OUT14)
- new net LAGER_L_L: LAGER_1_T_L1.24 (G), LAGER_2_T_L1.24 (G), LAGER_3_T_L1.24 (G), U6.15 (OUT15)
- new net LAGER_L_YD1: U6.1 (OUT1), YD19.1 (K), YD25.1 (K), YD31.1 (K)
- new net LAGER_L_YD2: U6.2 (OUT2), YD26.1 (K), YD32.1 (K)
- new net LAGER_L_YD3: U6.3 (OUT3), YD27.1 (K), YD33.1 (K)
- new net LAGER_R_A: LAGER_1_T_R1.2 (R), LAGER_2_T_R1.2 (R), LAGER_3_T_R1.2 (R), U7.4 (OUT4)
- new net LAGER_R_B: LAGER_1_T_R1.4 (R), LAGER_2_T_R1.4 (R), LAGER_3_T_R1.4 (R), U7.5 (OUT5)
- new net LAGER_R_C: LAGER_1_T_R1.6 (R), LAGER_2_T_R1.6 (R), LAGER_3_T_R1.6 (R), U7.6 (OUT6)
- new net LAGER_R_D: LAGER_1_T_R1.8 (R), LAGER_2_T_R1.8 (R), LAGER_3_T_R1.8 (R), U7.7 (OUT7)
- new net LAGER_R_E: LAGER_1_T_R1.10 (G), LAGER_2_T_R1.10 (G), LAGER_3_T_R1.10 (G), U7.8 (OUT8)
- new net LAGER_R_F: LAGER_1_T_R1.12 (G), LAGER_2_T_R1.12 (G), LAGER_3_T_R1.12 (G)
- new net LAGER_R_G: LAGER_1_T_R1.14 (G), LAGER_2_T_R1.14 (G), LAGER_3_T_R1.14 (G)
- new net LAGER_R_H: LAGER_1_T_R1.16 (G), LAGER_2_T_R1.16 (G), LAGER_3_T_R1.16 (G)
- new net LAGER_R_I: LAGER_1_T_R1.18 (G), LAGER_2_T_R1.18 (G), LAGER_3_T_R1.18 (G)
- new net LAGER_R_J: LAGER_1_T_R1.20 (G), LAGER_2_T_R1.20 (G), LAGER_3_T_R1.20 (G)
- new net LAGER_R_K: LAGER_1_T_R1.22 (G), LAGER_2_T_R1.22 (G), LAGER_3_T_R1.22 (G)
- new net LAGER_R_L: LAGER_1_T_R1.24 (G), LAGER_2_T_R1.24 (G), LAGER_3_T_R1.24 (G)
- new net SCLK_2: TTGO2.5 (GPIO25), U6.25 (SCLK), U7.25 (SCLK), U8.25 (SCLK), U9.25 (SCLK)
- new net SIG_6: TTGO2.6 (GPIO33), U6.26 (SIN)
- new net SIG_7: U6.17 (SOUT), U7.26 (SIN)
- new net SIG_8: U7.17 (SOUT), U8.26 (SIN)
- new net SIG_9: U8.17 (SOUT), U9.26 (SIN)
- new net SOUT_2: TTGO2.20 (GPIO13), U9.17 (SOUT)
- new net VPRG_2: TTGO2.7 (GPIO32), U6.27 (VPRG), U7.27 (VPRG), U8.27 (VPRG), U9.27 (VPRG)
- new net XLAT_2: TTGO2.4 (GPIO26), U6.24 (XLAT), U7.24 (XLAT), U8.24 (XLAT), U9.24 (XLAT)
- no-connect marks 35 -> 42
Other:
- moved on the sheet: C1, C12, C13, C2, C3, C4, C5, C6, C7, C8, C9, CG1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
